Commit message: Renombrado a sin 2027

File: description/robot.urdf.xacro (robot description, xacro)
@@ -1,4 +1,4 @@
 <?xml version="1.0"?>
-<robot xmlns:xacro="http://www.ros.org/wiki/xacro" name="eurobot2027">
+<robot xmlns:xacro="http://www.ros.org/wiki/xacro" name="eurobot">
     <xacro:include filename="robot_core.xacro" />
     <xacro:include filename="lidar.xacro" />

File: description/robot_core.xacro (robot description, xacro)
@@ -108,5 +108,5 @@
                 <origin xyz="0 0 0" rpy="0 0 ${rotacion_z}"/>                               <!-- No necesario ahora pero por si al importar el stl no encaja-->
                 <geometry>
-                    <cylinder radius="0.0325" length="0.04"/>                               <!-- <mesh filename="file://$(find eurobot2027_software_simulacion)/description/meshes/rueda.stl" scale="1 1 1"/> para cuando se añada el stl-->
+                    <cylinder radius="0.0325" length="0.04"/>                               <!-- <mesh filename="file://$(find eurobot_software_simulacion)/description/meshes/rueda.stl" scale="1 1 1"/> para cuando se añada el stl-->
                 </geometry>
                 <material name="blue"/>
